File: robot_sch/sch.kicad_pcb (KiCad board)
At the start: 2 copper layers, 46.1 x 34.7 mm, 21 parts, among them J1 Conn_01x04, J2 Conn_02x01, J3 Conn_02x04_Odd_Even, J4 Conn_02x01, J5 Conn_02x01, J6 Conn_01x04, J7 Conn_01x06, U1 STM32F103C8Tx, U2 AP1117-33

Commit message: nrf on 411 ok
Routing:
- net GND: track 81.4 -> 58.2 mm
- net +3V3: track 132.6 -> 131.7 mm
