File: robot_sch/sch.sch (KiCad schematic (older format))
At the start: 21 parts, among them J1 Conn_01x04, J2 Conn_02x01, J3 Conn_02x04_Odd_Even, J4 Conn_02x01, J5 Conn_02x01, J6 Conn_01x04, J7 Conn_01x06, U1 STM32F103C8Tx, U2 AP1117-33

Commit message: 6 pults ready
Parts:
- U1: symbol MCU_ST_STM32F1:STM32F103C8Tx -> sch-rescue:STM32F103C8Tx-MCU_ST_STM32F1
Changed lines of the file:
@@
 	7950 2600 8050 2600
 $Comp
-L power:+3.3V #PWR0101
+L sch-rescue:+3.3V-power #PWR0101
 U 1 1 5C096C9E
 P 7950 2550
@@
 $EndComp
 $Comp
-L power:GND #PWR0102
+L sch-rescue:GND-power #PWR0102
 U 1 1 5C096D17
 P 7950 3150
@@
 	7950 3100 8050 3100
 $Comp
-L power:GND #PWR0103
+L sch-rescue:GND-power #PWR0103
 U 1 1 5C096FD2
 P 4550 5200
@@
 	4700 2050 4600 2050
 $Comp
-L power:+3.3V #PWR0104
+L sch-rescue:+3.3V-power #PWR0104
 U 1 1 5C09A14A
 P 4600 2000
@@
 	4600 2000 4600 2050
 $Comp
-L power:GND #PWR0105
+L sch-rescue:GND-power #PWR0105
 U 1 1 5C09AC46
 P 7950 4800
@@
 	7950 4750 7900 4750
 $Comp
-L power:+3.3V #PWR0106
+L sch-rescue:+3.3V-power #PWR0106
 U 1 1 5C09B6FF
 P 7350 4800
@@
 $EndComp
 $Comp
-L power:GND #PWR0107
+L sch-rescue:GND-power #PWR0107
 U 1 1 5C0A4A65
 P 3250 2550
@@
 	6950 5500 7350 5500
 $Comp
-L power:GND #PWR0108
+L sch-rescue:GND-power #PWR0108
 U 1 1 5C0B768D
 P 7850 6200
@@
 	8350 6150 7850 6150
 $Comp
-L power:+3.3V #PWR0109
+L sch-rescue:+3.3V-power #PWR0109
 U 1 1 5C0C1827
 P 8350 5450
@@
 Connection ~ 8350 5500
 $Comp
-L power:GND #PWR0110
+L sch-rescue:GND-power #PWR0110
 U 1 1 5C0C37D2
 P 5800 5000
@@
 	5800 5000 5800 4900
 $Comp
-L power:+3.3V #PWR0111
+L sch-rescue:+3.3V-power #PWR0111
 U 1 1 5C0C79EF
 P 5950 5100
@@
 $EndComp
 $Comp
-L power:GND #PWR0112
+L sch-rescue:GND-power #PWR0112
 U 1 1 5C0C7B07
 P 6400 4650
@@
 $EndComp
 $Comp
-L MCU_ST_STM32F1:STM32F103C8Tx U1
+L sch-rescue:STM32F103C8Tx-MCU_ST_STM32F1 U1
 U 1 1 5C091EBB
 P 4600 3600
