File: sch/sch.kicad_pcb (KiCad board)
At the start: 2 copper layers, 46.1 x 34.7 mm, 22 parts, among them J1 Conn_01x04, J2 Conn_02x01, J3 Conn_02x04_Odd_Even, J4 Conn_02x01, SW1 SW_Push, U1 STM32F103C8Tx, U2 AP1117-33

Commit message: nrf on 411 ok
Routing:
- net GND: track 179.7 -> 113.9 mm
- net +3V3: track 135.2 -> 136.1 mm
- net /SWDIO: track 15.4 -> 14.7 mm
